Commit message: fix coordinate system

File: urdf/robot.urdf (robot description, URDF)
Before this commit: robot lidar_camera, 4 links, 3 joints
Links:
- removed link base_scan
- added link lidar
Joints:
- removed joint base_to_scan
- added joint base_to_lidar: type fixed, parent base_link, child lidar, origin xyz=0.0 0.0 -.003 rpy=0.0 0.0 0.0
- joint base_to_camera: origin xyz=0.11 0.015 0.065 rpy=1.57079 0.0 -1.57079 -> xyz=0.0 -0.135 -0.145 rpy=1.57079 0.0 1.57079
- joint camera_to_optical: origin xyz=0 0 0.02745 rpy=0 0 0 -> xyz=0.0 0 0.0 rpy=0 0 0
